Commit message: add 6

File: 5/ex03..05/minigun_resources/models/model.gazebo.xacro (robot description, xacro)
@@ -21,3 +21,71 @@
     </plugin>
   </gazebo>
+  <gazebo reference="lidar_frame">
+    <sensor name="gpu_lidar" type="gpu_lidar">
+      <topic>lidar</topic>
+      <gz_frame_id>lidar_frame</gz_frame_id>
+      <update_rate>10</update_rate>
+      <ray>
+        <scan>
+          <horizontal>
+            <samples>640</samples>
+            <resolution>1</resolution>
+            <min_angle>-1.396263</min_angle>
+            <max_angle>1.396263</max_angle>
+          </horizontal>
+          <vertical>
+            <samples>1</samples>
+            <resolution>0.01</resolution>
+            <min_angle>0</min_angle>
+            <max_angle>0</max_angle>
+          </vertical>
+        </scan>
+        <range>
+          <min>0.08</min>
+          <max>10.0</max>
+          <resolution>0.01</resolution>
+        </range>
+      </ray>
+      <always_on>1</always_on>
+      <visualize>true</visualize>
+    </sensor>
+  </gazebo>
+  <gazebo reference="depth_frame">
+    <sensor name="depth" type="depth_camera">
+      <topic>depth</topic>
+      <gz_frame_id>depth_frame</gz_frame_id>
+      <update_rate>6</update_rate>
+      <always_on>0</always_on>
+      <camera>
+        <horizontal_fov>1.51843645</horizontal_fov>
+        <image>
+          <width>848</width>
+          <height>480</height>
+          <format>R_FLOAT32</format>
+        </image>
+        <clip>
+          <near>0.1</near>
+          <far>10</far>
+        </clip>
+        <lens>
+          <intrinsics>
+            <fx>421.61578369140625</fx>
+            <fy>421.61578369140625</fy>
+            <cx>422.2854309082031</cx>
+            <cy>236.57237243652344</cy>
+            <s>0</s>
+          </intrinsics>
+        </lens>
+      </camera>
+    </sensor>
+  </gazebo>
+  <gazebo reference="frame">
+    <sensor name="imu_sensor" type="imu">
+      <gz_frame_id>frame</gz_frame_id>
+      <always_on>1</always_on>
+      <update_rate>60</update_rate>
+      <visualize>true</visualize>
+      <topic>imu</topic>
+    </sensor>
+  </gazebo>
 </robot>

File: 5/ex03..05/minigun_resources/models/model.urdf.xacro (robot description, xacro)
@@ -141,3 +141,15 @@
     <axis xyz="1 0 0" />
   </joint>
+  <link name="lidar_frame" />
+  <joint name="lidar_frame_joint" type="fixed">
+    <parent link="frame" />
+    <child link="lidar_frame" />
+    <origin xyz="0 ${-5.5*s} ${0*s}" rpy="0 0 ${-pi/2}" />
+  </joint>
+  <link name="depth_frame" />
+  <joint name="depth_frame_joint" type="fixed">
+    <parent link="frame" />
+    <child link="depth_frame" />
+    <origin xyz="0 ${-5.5*s} ${0*s}" rpy="0 0 ${-pi/2}" />
+  </joint>
 </robot>
